Commit message: Activity 04

File: second-ws/src/my_robot_description/urdf/common_properties.xacro (robot description, xacro)
@@ -7,3 +7,30 @@
         <color rgba="0.5 0.5 0.5 1" />
     </material>
+    <xacro:macro name="box_inertial" params="m l w h xyz rpy">
+        <inertial>
+            <origin xyz="${xyz}" rpy="${rpy}"/>
+            <mass value="${m}" />
+            <interia ixx="${(m/12) * (h*h + l*l)}" ixy="0" ixz="0"
+                     iyy="${(m/12) * (w*w + l*l)}" iyz ="0"
+                     izz="${(m/12) * (w*w + h*h)}" />
+        </inertial>
+    </xacro:macro>
+    <xacro:macro name="sphere_inertial" params="m r xyz rpy">
+        <inertial>
+            <origin xyz="${xyz}" rpy="${rpy}"/>
+            <mass value="${m}" />
+            <interia ixx="${(2/5) * m * r*r}" ixy="0" ixz="0"
+                     iyy="${(2/5) * m * r*r}" iyz ="0"
+                     izz="${(2/5) * m * r*r}" />
+        </inertial>
+    </xacro:macro>
+    <xacro:macro name="cylinder_inertial" params="m r h xyz rpy">
+        <inertial>
+            <origin xyz="${xyz}" rpy="${rpy}"/>
+            <mass value="${m}" />
+            <interia ixx="${(m/12) * (3*r*r + h*h)}" ixy="0" ixz="0"
+                     iyy="${(m/12) * (3*r*r + h*h)}" iyz ="0"
+                     izz="${(m/2) * m * r*r}" />
+        </inertial>
+    </xacro:macro>
 </robot>

File: second-ws/src/my_robot_description/urdf/mobile_base.xacro (robot description, xacro)
@@ -15,4 +15,5 @@
                 <material name="grey" />
             </visual>
+            <xacro:sphere_interia m="1.0" r="${wheel_radius}" h="${wheel_length}" xyz="0 0 0" rpy="${pi / 2.0} 0 0"/>
         </link>
     </xacro:macro>
@@ -28,4 +29,5 @@
             <material name="blue" />
         </visual>
+        <xacro:box_interia m="5.0" l="${base_length}" w="${base_width}" h="${base_height}" xyz="0 0 ${base_height / 2}" rpy="0 0 0"/>
     </link>
     <link name="caster_wheel_link">
@@ -37,4 +39,5 @@
             <material name="grey" />
         </visual>
+        <xacro:sphere_interia m="0.5" r="${wheel_radius}" xyz="0 0 0" rpy="0 0 0"/>
     </link>
     <joint name="base_joint" type="fixed">

Commit message: Spawn my_robot in gazebo

File: second-ws/src/my_robot_description/urdf/common_properties.xacro (robot description, xacro)
@@ -7,29 +7,29 @@
         <color rgba="0.5 0.5 0.5 1" />
     </material>
-    <xacro:macro name="box_inertial" params="m l w h xyz rpy">
+    <xacro:macro name="box_inertia" params="m l w h xyz rpy">
         <inertial>
-            <origin xyz="${xyz}" rpy="${rpy}"/>
+            <origin xyz="${xyz}" rpy="${rpy}" />
             <mass value="${m}" />
-            <interia ixx="${(m/12) * (h*h + l*l)}" ixy="0" ixz="0"
-                     iyy="${(m/12) * (w*w + l*l)}" iyz ="0"
+            <inertia ixx="${(m/12) * (h*h + l*l)}" ixy="0" ixz="0"
+                     iyy="${(m/12) * (w*w + l*l)}" iyz="0"
                      izz="${(m/12) * (w*w + h*h)}" />
         </inertial>
     </xacro:macro>
-    <xacro:macro name="sphere_inertial" params="m r xyz rpy">
+    <xacro:macro name="cylinder_inertia" params="m r h xyz rpy">
         <inertial>
-            <origin xyz="${xyz}" rpy="${rpy}"/>
+            <origin xyz="${xyz}" rpy="${rpy}" />
             <mass value="${m}" />
-            <interia ixx="${(2/5) * m * r*r}" ixy="0" ixz="0"
-                     iyy="${(2/5) * m * r*r}" iyz ="0"
-                     izz="${(2/5) * m * r*r}" />
+            <inertia ixx="${(m/12) * (3*r*r + h*h)}" ixy="0" ixz="0"
+                     iyy="${(m/12) * (3*r*r + h*h)}" iyz="0"
+                     izz="${(m/2) * (r*r)}" />
         </inertial>
     </xacro:macro>
-    <xacro:macro name="cylinder_inertial" params="m r h xyz rpy">
+    <xacro:macro name="sphere_inertia" params="m r xyz rpy">
         <inertial>
-            <origin xyz="${xyz}" rpy="${rpy}"/>
+            <origin xyz="${xyz}" rpy="${rpy}" />
             <mass value="${m}" />
-            <interia ixx="${(m/12) * (3*r*r + h*h)}" ixy="0" ixz="0"
-                     iyy="${(m/12) * (3*r*r + h*h)}" iyz ="0"
-                     izz="${(m/2) * m * r*r}" />
+            <inertia ixx="${(2/5) * m * r * r}" ixy="0" ixz="0"
+                     iyy="${(2/5) * m * r * r}" iyz="0"
+                     izz="${(2/5) * m * r * r}" />
         </inertial>
     </xacro:macro>

File: second-ws/src/my_robot_description/urdf/mobile_base.xacro (robot description, xacro)
@@ -6,4 +6,16 @@
     <xacro:property name="wheel_radius" value="0.1" />
     <xacro:property name="wheel_length" value="0.05" />
+    <link name="base_footprint" />
+    <link name="base_link">
+        <visual>
+            <geometry>
+                <box size="${base_length} ${base_width} ${base_height}" />
+            </geometry>
+            <origin xyz="0 0 ${base_height / 2.0}" rpy="0 0 0" />
+            <material name="blue" />
+        </visual>
+        <xacro:box_inertia m="5.0" l="${base_length}" w="${base_width}" h="${base_height}"
+                           xyz="0 0 ${base_height / 2.0}" rpy="0 0 0" />
+    </link>
     <xacro:macro name="wheel_link" params="prefix">
         <link name="${prefix}_wheel_link">
@@ -15,29 +27,20 @@
                 <material name="grey" />
             </visual>
-            <xacro:sphere_interia m="1.0" r="${wheel_radius}" h="${wheel_length}" xyz="0 0 0" rpy="${pi / 2.0} 0 0"/>
+            <xacro:cylinder_inertia m="1.0" r="${wheel_radius}" h="${wheel_length}"
+                                    xyz="0 0 0" rpy="${pi / 2.0} 0 0" />
         </link>
     </xacro:macro>
-    <xacro:wheel_link prefix="right"/>
-    <xacro:wheel_link prefix="left"/>
-    <link name="base_footprint" />
-    <link name="base_link">
-        <visual>
-            <geometry>
-                <box size="${base_length} ${base_width} ${base_height}" />
-            </geometry>
-            <origin xyz="0 0 ${base_height / 2}" rpy="0 0 0" />
-            <material name="blue" />
-        </visual>
-        <xacro:box_interia m="5.0" l="${base_length}" w="${base_width}" h="${base_height}" xyz="0 0 ${base_height / 2}" rpy="0 0 0"/>
-    </link>
+    <xacro:wheel_link prefix="right" />
+    <xacro:wheel_link prefix="left" />
     <link name="caster_wheel_link">
         <visual>
             <geometry>
-                <sphere radius="${wheel_radius}" />
+                <sphere radius="${wheel_radius / 2.0}" />
             </geometry>
             <origin xyz="0 0 0" rpy="0 0 0" />
             <material name="grey" />
         </visual>
-        <xacro:sphere_interia m="0.5" r="${wheel_radius}" xyz="0 0 0" rpy="0 0 0"/>
+        <xacro:sphere_inertia m="0.5" r="${wheel_radius / 2.0}"
+                              xyz="0 0 0" rpy="0 0 0" />
     </link>
     <joint name="base_joint" type="fixed">
@@ -49,5 +52,5 @@
         <parent link="base_link" />
         <child link="right_wheel_link" />
-        <origin xyz="${-base_lenght / 4.0} ${-(base_width + wheel_length) / 2.0} 0" rpy="0 0 0" />
+        <origin xyz="${-base_length / 4.0} ${-(base_width + wheel_length) / 2.0} 0" rpy="0 0 0" />
         <axis xyz="0 1 0" />
     </joint>
@@ -55,5 +58,5 @@
         <parent link="base_link" />
         <child link="left_wheel_link" />
-        <origin xyz="${-base_lenght / 4.0} ${(base_width + wheel_length) / 2.0} 0" rpy="0 0 0" />
+        <origin xyz="${-base_length / 4.0} ${(base_width + wheel_length) / 2.0} 0" rpy="0 0 0" />
         <axis xyz="0 1 0" />
     </joint>
@@ -61,5 +64,5 @@
         <parent link="base_link" />
         <child link="caster_wheel_link" />
-        <origin xyz="${base_lenght / 3.0} 0 ${-wheel_radius / 2}" rpy="0 0 0" />
+        <origin xyz="${base_length / 3.0} 0 ${-wheel_radius / 2.0}" rpy="0 0 0" />
     </joint>
 </robot>
